File: hardware/boards/daisyBoard.kicad_sch (KiCad schematic)
At the start: 59 parts, among them IC1 TL072, IC2 TL072, IC3 TL072, IC4 TL072, J1 LEFT Pin ROW, J10 AudioJack_OUT_2, J11 AudioJack_OUT_2, J2 RIGHT Pin Row, J5 Micro_SD_Card, J6 AudioJack3, J7 AudioJack3, J8 AudioJack_IN_1, J9 AudioJack_IN_2, U3 MCP6002-xMC, U4 MCP6002-xMC

Commit message: changes
Parts:
- added C14: 0.1uF, symbol Device:C
- added C18: 10uF, symbol Device:C
- added J12: Micro_SD_Card, symbol Connector:Micro_SD_Card
- added R25, R26, R27: 10K, Resistor_SMD:R_0805_2012Metric, symbol Device:R
Connections:
- net GND: now also C14.1, C18.1, J12.6 (VSS), J12.SH (SHIELD)
- net SD_MOSI: now reaches J2.1 (Pin_1)
- net SD_MOSI: now also J12.3 (CMD), R26.2
- net ESP-3.3V: now reaches J2.15 (Pin_15)
- net ESP-3.3V: now also C14.2, C18.2, J12.4 (VDD), R25.1, R26.1, R27.1
- net SD_MISO: now reaches J2.6 (Pin_6)
- net SD_MISO: now also J12.7 (DAT0), R27.2
- net SD_SCK: now reaches J2.7 (Pin_7)
- net SD_SCK: now also J12.5 (CLK)
- net SD_CS: now reaches J2.8 (Pin_8)
- net SD_CS: now also J12.2 (DAT3/CD), R25.2
- no-connect marks 4 -> 6
Other:
- note added: "Decoup Caps close to VDD input"
- note added: "SD CARD INTERFACE DAISY"
- note removed: "SD CARD INTERFACE"

Commit message: Intermediate update
Parts:
- removed A1: Electrosmith_Daisy_Seed_Rev4, Module:Electrosmith_Daisy_Seed, symbol MCU_Module:Electrosmith_Daisy_Seed_Rev4
- removed D2, D3: 1N5817, Diode_SMD:D_SMF, symbol Diode:1N5817
- removed U3, U4: MCP6002-xMC, Package_DFN_QFN:DFN-8-1EP_3x2mm_P0.5mm_EP1.75x1.45mm, symbol Amplifier_Operational:MCP6002-xMC
- removed V2: VSIN, symbol Simulation_SPICE:VSIN
- added C20, C22, C23: 100n, Capacitor_SMD:C_1206_3216Metric, symbol Device:C
- added C21: 100u, Capacitor_SMD:C_1206_3216Metric, symbol Device:C_Polarized_US
- added FB1, FB2, FB3: 600R @ 100MHz, Inductor_SMD:L_0805_2012Metric, symbol Device:FerriteBead
- added unit 2 of IC1
- added unit 2 of IC2
- added unit 2 of IC3
- added unit 2 of IC4
- added J13: LEFT Pin ROW Daisy, Connector_PinSocket_2.54mm:PinSocket_1x20_P2.54mm_Vertical, symbol Connector:Conn_01x20_Pin
- added J14: RIGHT Pin ROW DAISY, Connector_PinSocket_2.54mm:PinSocket_1x20_P2.54mm_Vertical, symbol Connector:Conn_01x20_Pin
- added J15: Daisy Pin Breakout LEFT, Connector_PinHeader_2.54mm:PinHeader_1x20_P2.54mm_Vertical, symbol Connector:Conn_01x20_Pin
- added J16: Daisy PIN Breakout RIGHT, Connector_PinHeader_2.54mm:PinHeader_1x20_P2.54mm_Vertical, symbol Connector:Conn_01x20_Pin
- added J3: ESP32 Pin Breakout RIGHT, Connector_PinHeader_2.54mm:PinHeader_1x15_P2.54mm_Vertical, symbol Connector:Conn_01x15_Pin
- added J4: ESP32 Pin Breakout LEFT, Connector_PinHeader_2.54mm:PinHeader_1x15_P2.54mm_Vertical, symbol Connector:Conn_01x15_Pin
- added NT1: NetTie_2, NetTie:NetTie-2_SMD_Pad0.5mm, symbol Device:NetTie_2
- added R24: 100R, Resistor_SMD:R_0805_2012Metric, symbol Device:R
- added TP1: Global Ground - Functional, TestPoint:TestPoint_THTPad_D2.5mm_Drill1.2mm, symbol Connector:TestPoint
- added TP10: Jack Input 1 Pad GND, TestPoint:TestPoint_THTPad_D2.5mm_Drill1.2mm, symbol Connector:TestPoint
- added TP11: Jack Output 2 Signal Pad, TestPoint:TestPoint_THTPad_D2.5mm_Drill1.2mm, symbol Connector:TestPoint
- added TP12: Jack Output 2 GND Pad, TestPoint:TestPoint_THTPad_D2.5mm_Drill1.2mm, symbol Connector:TestPoint
- added TP15: Jack Output 1 GND Pad, TestPoint:TestPoint_THTPad_D2.5mm_Drill1.2mm, symbol Connector:TestPoint
- added TP16: Jack Output 1 Signal Pad, TestPoint:TestPoint_THTPad_D2.5mm_Drill1.2mm, symbol Connector:TestPoint
- added TP17: Exp Jack Input 1 Pad GND, TestPoint:TestPoint_THTPad_D2.5mm_Drill1.2mm, symbol Connector:TestPoint
- added TP18: Exp Jack Input 1 Signal, TestPoint:TestPoint_THTPad_D2.5mm_Drill1.2mm, symbol Connector:TestPoint
- added TP19: Exp Jack Input 2 GND, TestPoint:TestPoint_THTPad_D2.5mm_Drill1.2mm, symbol Connector:TestPoint
- added TP2: Global power 5V Input field - Functional, TestPoint:TestPoint_THTPad_D2.5mm_Drill1.2mm, symbol Connector:TestPoint
- added TP20: Exp Jack Input 2 Signal, TestPoint:TestPoint_THTPad_D2.5mm_Drill1.2mm, symbol Connector:TestPoint
- added TP21: Processed input power at 5V ESP32 - Probe, TestPoint:TestPoint_Pad_2.0x2.0mm, symbol Connector:TestPoint
- added TP22: EXPR REF 1, TestPoint:TestPoint_THTPad_D2.5mm_Drill1.2mm, symbol Connector:TestPoint
- added TP23: EXPR Ref 2, TestPoint:TestPoint_THTPad_D2.5mm_Drill1.2mm, symbol Connector:TestPoint
- added TP5: Reference voltage for the op amps - Probe, TestPoint:TestPoint_Pad_2.0x2.0mm, symbol Connector:TestPoint
- added TP6: Processed input power at 5V Daisy- Probe, TestPoint:TestPoint_Pad_2.0x2.0mm, symbol Connector:TestPoint
- added TP7: Jack Input 1 Pad, TestPoint:TestPoint_THTPad_D2.5mm_Drill1.2mm, symbol Connector:TestPoint
- added TP8: Jack Input 2 Pad, TestPoint:TestPoint_THTPad_D2.5mm_Drill1.2mm, symbol Connector:TestPoint
- added TP9: Jack Input 2 Pad GND, TestPoint:TestPoint_THTPad_D2.5mm_Drill1.2mm, symbol Connector:TestPoint
- added U1, U2, U3: MCP6002-xSN, Package_SO:SOIC-8_3.9x4.9mm_P1.27mm, symbol Amplifier_Operational:MCP6002-xSN
- C1: footprint Capacitor_SMD:C_0201_0603Metric -> Capacitor_SMD:C_1206_3216Metric
- C10, C11, C12, C13, C14, C15, C16, C17, C18, C19, C2, C3, C4, C5, C6, C7, C8, C9: footprint (none) -> Capacitor_SMD:C_1206_3216Metric
- IC1, IC2, IC3, IC4: footprint (none) -> Package_SO:SOIC-8_3.9x4.9mm_P1.27mm
- J10, J11, J6, J7, J8, J9: now left out of the parts list
- J12, J5: footprint (none) -> Connector_Card:microSD_HC_Molex_104031-0811
- R13, R14, R15, R16, R17: value 47K -> 10K
Connections:
- net +3.3VA: now also J13.20 (Pin_20), J15.1 (Pin_1), U1.3 (+), U2.3 (+)
- net +3.3VD: now also J13.3 (Pin_3), J15.18 (Pin_18)
- net +5V: now also FB1.1, NT1.1, TP2.1, U3.8 (V+); no longer C15.1
- net ADC_EXP_IN_1: now also J13.18 (Pin_18), J15.3 (Pin_3), U1.6 (-), U1.7
- net ADC_EXP_IN_2: now also J13.19 (Pin_19), J15.2 (Pin_2), U2.6 (-), U2.7
- net AUDIO_IN_1: now also J14.5 (Pin_5), J16.16 (Pin_16)
- net AUDIO_IN_2: now also J14.4 (Pin_4), J16.17 (Pin_17)
- net AUDIO_OUT_1: now also J14.3 (Pin_3), J16.18 (Pin_18); no longer R9.2
- net AUDIO_OUT_2: now also R9.2, J14.2 (Pin_2), J16.19 (Pin_19)
- net DAISY_TO_ESP: now also J2.10 (Pin_10), J14.7 (Pin_7), J16.14 (Pin_14), J3.6 (Pin_6); no longer J2.4 (Pin_4)
- net ESP-3.3V: now also J3.1 (Pin_1)
- net ESP_TO_DAISY: now also J2.9 (Pin_9), J14.6 (Pin_6), J16.15 (Pin_15), J3.7 (Pin_7); no longer J2.3 (Pin_3)
- net EXPRESSION_REF: no longer R18.2, R21.2
- net GND: now also FB2.2, FB3.2, TP1.1; no longer C1.2, C10.2, C13.2, C14.1, C15.2, C16.2, C17.2, C18.1, C19.2, C3.1, C4.2, C6.1, C7.2, IC1.4 (V-), IC2.4 (V-), IC3.4 (V-), IC4.4 (V-), J1.2 (Pin_2), J10.S, J11.S, J12.6 (VSS), J12.SH (SHIELD), J2.14 (Pin_14), J5.6 (VSS), J5.SH (SHIELD), J6.S, J7.S, J8.S, J9.S, R12.2, R19.2, R20.2, R23.1, R8.2
- net SD_CLK_DAISY: now also J14.14 (Pin_14), J16.7 (Pin_7)
- net SD_CMD_DAISY: now also J14.15 (Pin_15), J16.6 (Pin_6)
- net SD_CS: now also J3.8 (Pin_8)
- net SD_DAT_0_DAISY: now also J14.16 (Pin_16), J16.5 (Pin_5)
- net SD_DAT_1_DAISY: now also J14.17 (Pin_17), J16.4 (Pin_4)
- net SD_DAT_2_DAISY: now also J14.18 (Pin_18), J16.3 (Pin_3)
- net SD_DAT_3_DAISY: now also J14.19 (Pin_19), J16.2 (Pin_2)
- net SD_MISO: now also J3.10 (Pin_10)
- net SD_MOSI: now also J3.15 (Pin_15)
- net SD_SCK: now also J3.9 (Pin_9)
- net VREF: now also R24.2, TP5.1, U3.2 (-); no longer C19.1, R22.1, R23.2
- net at J7.T, R20.1: now also TP20.1, U2.5 (+)
- net at C12.2, J10.T, R12.1: now also TP11.1
- net at C8.2, R6.2: now also IC3.3 (+)
- net at R21.1: now also U2.1, U2.2 (-)
- net at C9.2, J11.T, R8.1: now also TP16.1
- net at C4.1, C5.1, J9.T: now also TP8.1
- net at C1.1, C2.1, J8.T: now also TP7.1
- net VCC_ESP32: now reaches J1.1 (Pin_1)
- net VCC_ESP32: now also C21.1, C22.1, C23.1, FB1.2, J4.15 (Pin_15), TP21.1
- net at J1.10 (Pin_10): now also J4.6 (Pin_6)
- net at J1.11 (Pin_11): now also J4.5 (Pin_5)
- net at J1.12 (Pin_12): now also J4.4 (Pin_4)
- net at J1.13 (Pin_13): now also J4.3 (Pin_3)
- net at J1.14 (Pin_14): now also J4.2 (Pin_2)
- net at J1.15 (Pin_15): now also J4.1 (Pin_1)
- net at J1.3 (Pin_3): now also J4.13 (Pin_13)
- net at J1.4 (Pin_4): now also J4.12 (Pin_12)
- net at J1.5 (Pin_5): now also J4.11 (Pin_11)
- net at J1.6 (Pin_6): now also J4.10 (Pin_10)
- net at J1.7 (Pin_7): now also J4.9 (Pin_9)
- net at J1.8 (Pin_8): now also J4.8 (Pin_8)
- net at J1.9 (Pin_9): now also J4.7 (Pin_7)
- net EXPRESSION_REF_1: now reaches R18.1
- net EXPRESSION_REF_1: now also TP22.1
- net at J6.T, R19.1: now also TP18.1, U1.5 (+)
- net at J2.11 (Pin_11): now also J3.5 (Pin_5)
- net at J2.12 (Pin_12): now also J3.4 (Pin_4)
- net at J2.13 (Pin_13): now also J3.3 (Pin_3)
- net at J2.2 (Pin_2): now also J3.14 (Pin_14)
- net at J2.5 (Pin_5): now also J3.11 (Pin_11)
- net VCC renamed VCC_Daisy
- net VCC_Daisy: now also J13.2 (Pin_2), J15.19 (Pin_19), NT1.2, TP6.1, U1.8 (V+), U2.8 (V+)
- new net: R24.1, U3.1
- new net: C15.1, C19.1, C20.1, R22.1, R23.2, U3.3 (+)
- new net: J13.10 (Pin_10), J15.11 (Pin_11)
- new net: J13.11 (Pin_11), J15.10 (Pin_10)
- new net: J13.12 (Pin_12), J15.9 (Pin_9)
- new net: J13.13 (Pin_13), J15.8 (Pin_8)
- new net: J13.14 (Pin_14), J15.7 (Pin_7)
- new net: J13.15 (Pin_15), J15.6 (Pin_6)
- new net: J13.16 (Pin_16), J15.5 (Pin_5)
- new net: J13.17 (Pin_17), J15.4 (Pin_4)
- new net: J13.4 (Pin_4), J15.17 (Pin_17)
- new net: J13.5 (Pin_5), J15.16 (Pin_16)
- new net: J13.6 (Pin_6), J15.15 (Pin_15)
- new net: J13.7 (Pin_7), J15.14 (Pin_14)
- new net: J13.8 (Pin_8), J15.13 (Pin_13)
- new net: J13.9 (Pin_9), J15.12 (Pin_12)
- new net: J14.10 (Pin_10), J16.11 (Pin_11)
- new net: J14.11 (Pin_11), J16.10 (Pin_10)
- new net: J14.12 (Pin_12), J16.9 (Pin_9)
- new net: J14.13 (Pin_13), J16.8 (Pin_8)
- new net: J14.20 (Pin_20), J16.1 (Pin_1)
- new net: J14.8 (Pin_8), J16.13 (Pin_13)
- new net: J14.9 (Pin_9), J16.12 (Pin_12)
- new net: R18.2, U1.1, U1.2 (-)
- new net: J2.4 (Pin_4), J3.12 (Pin_12)
- new net: J2.3 (Pin_3), J3.13 (Pin_13)
- new net EXPRESSION_REF_2: R21.2, TP23.1
- new net GNDA: C1.2, C10.2, C13.2, C15.2, C16.2, C17.2, C19.2, C20.2, C3.1, C4.2, C6.1, C7.2, FB2.1, IC1.4 (V-), IC2.4 (V-), IC3.4 (V-), IC4.4 (V-), J10.S, J11.S, J13.1 (Pin_1), J14.1 (Pin_1), J15.20 (Pin_20), J16.20 (Pin_20), J5.6 (VSS), J5.SH (SHIELD), J6.S, J7.S, J8.S, J9.S, R12.2, R19.2, R20.2, R23.1, R8.2, TP10.1, TP12.1, TP15.1, TP17.1, TP19.1, TP9.1, U1.4 (V-), U2.4 (V-), U3.4 (V-)
- new net GNDD: C14.1, C18.1, C21.2, C22.2, C23.2, FB3.1, J1.2 (Pin_2), J12.6 (VSS), J12.SH (SHIELD), J2.14 (Pin_14), J3.2 (Pin_2), J4.14 (Pin_14)
- no-connect marks 6 -> 24
Other:
- note added: "- Connector: USB - C - Voltage: 5.0 VDC (Nominal) - Current: A 3A (Often max current draw on premade breakout boards)"
- note added: "Buffered VREF"
- note added: "DAISY SEED"
- note added: "Daisy Power"
- note added: "Esp32 Power"
- note added: "Functional probes are better THT. While Probe is better with a pad"
- note added: "GND Seperation"
- note added: "Place these two next to eachother"
- note added: "Power Pads"
- note added: "Probes are purely for diagnostic purposes. Funcional can be used to power or transmit signals and add functionality"
- note added: "SD CARD INTERFACE ESP32"
- note added: "Solderpads/ Test Probes"
- note added: "USB Side"
- note added: "Voltage devider"
- note removed: "+5V Coming from prebuilt usb C breakout board BREAKOUT BOARD ALSO CONTAINS THE MAIN GND TERMINAL"
- note removed: "- Connector: USB - C - Voltage: 5.0 VDC (Nominal) - Current: A 5A (Often max current draw on premade breakout boards)"
- note removed: "Chosen Component Notes"
- note removed: "LM1117T-3.3 : Voltage Regulator rated up to 800mA (might need to change to high amperage buck converter depending on the peripheral used)"
- moved on the sheet: C1, C10, C11, C12, C13, C16, C17, C19, C2, C3, C4, C5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
